File: CharliesAlienWhoopF4.sch (EAGLE design)
At the start: 41 parts, among them M1 53047-0210, M2 53047-0210, M3 53047-0210, M4 53047-0210, Q1 FDMA410NZ, Q2 FDMA410NZ, Q3 IRLML6402, Q4 FDMA410NZ, Q5 FDMA410NZ, U1 MPU-9250, U2 TPS63001, Y1 8mhz

Commit message: I was having issues with solder bridges underneath the buckboost. Turns out my traces were too wide and when translated into gerber were leaving not much room for error. Hoping this makes reflow success rate 100% ;)
Connections:
- net N$7 renamed L1
- net N$8 renamed L2
Changed lines of the file:
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@@
 <?xml version="1.0" encoding="utf-8"?>
 <!DOCTYPE eagle SYSTEM "eagle.dtd">
-<eagle version="8.0.1">
+<eagle version="8.1.0">
 <drawing>
 <settings>
@@
 </segment>
 </net>
-<net name="N$7" class="0">
+<net name="L1" class="0">
 <segment>
 <pinref part="L1" gate="G$1" pin="1"/>
@@
 </segment>
 </net>
-<net name="N$8" class="0">
+<net name="L2" class="0">
 <segment>
 <pinref part="L1" gate="G$1" pin="2"/>
